File: Electronica/V1/shield_pi/shield_pi.kicad_pcb (KiCad board)
At the start: 2 copper layers, 65 x 56 mm, 7 parts, among them J1 GPIO, U2 TMC2209_SILENTSTEPSTICK, U3 TMC2209_SILENTSTEPSTICK

Commit message: prueba
Parts:
- moved U2 4.25 mm to (112.4, 64.1)
- moved U3 1.75 mm to (132.2, 64.1)
Changed lines of the file:
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@@
 	(footprint "TMC2209_SILENTSTEPSTICK:MODULE_TMC2209_SILENTSTEPSTICK"
 		(layer "F.Cu")
-		(at 116.605 64.11)
+		(at 112.355 64.11)
 		(property "Reference" "U2"
 			(at -5.075 -11.155 0)
@@
 		)
 		(property "Value" "TMC2209_SILENTSTEPSTICK"
-			(at 11.05 11.115 0)
+			(at 13.55 11.115 0)
 			(layer "F.Fab")
 			(effects
@@
 	(footprint "TMC2209_SILENTSTEPSTICK:MODULE_TMC2209_SILENTSTEPSTICK"
 		(layer "F.Cu")
-		(at 133.9 64.11)
+		(at 132.15 64.11)
 		(property "Reference" "U3"
 			(at -5.075 -11.155 0)
