File: Electronica/V1/shield_pi/shield_pi.kicad_sch (KiCad schematic)
At the start: 6 parts, among them J1 GPIO, U1 CAT24C256

Commit message: prueba
Parts:
- added U2, U3: TMC2209_SILENTSTEPSTICK, TMC2209_SILENTSTEPSTICK:MODULE_TMC2209_SILENTSTEPSTICK, symbol TMC2209_SILENTSTEPSTICK:TMC2209_SILENTSTEPSTICK
Connections:
- new net: U3.1 (GND), U3.7 (GND)
- new net: U2.1 (GND), U2.7 (GND)
